Commit message: Teil-A-Inbetriebnahme: RS485-Basisantrieb, VL53 über CH341A, RViz-Dummy
- base_hardware: pymodbus 3.x nutzt device_id= (statt slave/unit); invert_right
  auf false (ESS23-RS ignoriert das Register – Drehrichtung via Pr0.03 offen)
- vl53_near_field: VL53L5CX-Treiber-Chunk auf 32 reduziert (CH341-USB-I2C-Limit,
  sonst EIO im init), CH341-Busnummer dynamisch (i2c_bus_num: -1 -> _find_ch341_bus),
  Konstruktor-Multi-Signatur (bus_id=/i2c_bus=)
- robot_description: dummy_view.rviz (RobotModel+TF-Ansicht für display_dummy)
- übrige Config-/Doku-Änderungen aus dem Inbetriebnahme-Arbeitsstand
  (Prüfplan, READMEs, robot.launch.py, Gesicht-Web-UI, base_hardware-Params)

Stray-Klon src/BehaviorTree.ROS2/ bewusst nicht committet (dupliziert das
Submodul src/behaviortree_ros2, lokal per COLCON_IGNORE stillgelegt).

Co-Authored-By: Claude Opus 4.8 <noreply@anthropic.com>

File: src/robot_description/urdf/mobile_manipulator_dummy.urdf.xacro (robot description, xacro)
@@ -32,7 +32,9 @@
        wheel_separation = Abstand linker/rechter Radmittelpunkt.
        ================================================================ -->
-  <xacro:property name="wheel_radius"     value="0.075"/>
-  <xacro:property name="wheel_width"      value="0.040"/>
-  <xacro:property name="wheel_separation" value="0.420"/>
+  <!-- [GEMESSEN 13.07.2026] MUSS mit base_hardware_params.yaml uebereinstimmen! -->
+  <xacro:property name="wheel_radius"     value="0.0625"/>  <!-- Ø 125 mm -->
+  <xacro:property name="wheel_width"      value="0.040"/>   <!-- [ANPASSEN] -->
+  <xacro:property name="wheel_separation" value="0.378"/>   <!-- Radmitte-Radmitte -->
+  <!-- Getriebe 10:1 steht in base_hardware_params.yaml (gear_ratio) -->
   <xacro:property name="wheel_x"          value="0.000"/>
   <!-- ================================================================

Commit message: OAK-Tiefenkamera einbinden: Montagepose, TF unter base_link, schlanke Punktwolke
Bindet die OAK (aktuell Luxonis OAK-D-S2) als Projekt-Sensor ein - Grundlage
fuer vorausschauende Hindernisvermeidung, die mit den VL53 (50 cm) nicht geht.

- launch/oak.launch.py: startet depthai_ros_driver MIT der realen Montagepose,
  so dass der Treiber seine TF-Kette direkt unter base_link haengt (kein
  separater static_transform_publisher). Montagepose steht als einziger,
  klar markierter Block oben in der Datei.
- config/oak_params.yaml: Treibereinstellungen fuer den Costmap-Zweck
  (kein NN, HIGH_ACCURACY, Speckle-Filter, ISP-Skalierung auf 320x180).
- URDF: OAK-Pose auf die gemessenen Werte + Neigung (bisher Platzhalter ohne
  pitch): x=0.150, y=0, z=1.250 ueber base_link (=1.340 ueber Boden),
  20 Grad nach unten. Verifiziert: TF-Blickrichtung 20.0 Grad NACH UNTEN,
  optische Achse trifft den Boden bei 3.83 m.

Punktwolke bewusst mit depth_image_proc::PointCloudXyz (Tiefe + camera_info)
statt dem PointCloudXyzi aus depthai's pointcloud.launch.py: jenes braucht
/oak/right/image_rect, das an der MONO-Aufloesung haengt und nicht mit der
ISP-Groesse von RGB/Tiefe mitskaliert -> bei 320x180 Tiefe gegen 1280x720
Intensitaet entstanden voellig falsche 3D-Punkte (Punkte 5 m seitlich bei 2 m
Tiefe, Reichweiten bis -10 m). Jetzt entkoppelt, leichter, spart Bandbreite.

Gemessen nachher: 57.600 Punkte (48.824 gueltig) @7.8 Hz, Reichweite
0.93-11.27 m, 4.7 % Bodenpunkte - deckt sich mit der 720p-Referenzmessung
(4.6 %), 16x weniger Punkte als die 921.600er Rohwolke.

Weitere Fallstricke dokumentiert (alle real getestet): eine eigene params_file
ERSETZT depthai's pcl.yaml; ein fuer den IMX378 ungueltiges rgb.i_resolution
("720P") legt den RGB-Stream und damit die Wolke lahm.

Kamerawechsel auf OAK 4 D Pro Wide FF: Modell wird automatisch erkannt,
Vorlage liegt unter depthai_ros_driver/config/oak_d_pro_w.yaml.

Co-Authored-By: Claude Opus 4.8 <noreply@anthropic.com>

File: src/robot_description/urdf/mobile_manipulator_dummy.urdf.xacro (robot description, xacro)
@@ -39,11 +39,20 @@
   <xacro:property name="wheel_x"          value="0.000"/>
   <!-- ================================================================
-       SENSOR-MONTAGE: OAK 4 D PRO WIDE FF [ANPASSEN]
+       SENSOR-MONTAGE: OAK-Tiefenkamera
        camera_link ist mechanisch. camera_rgb_optical_frame ist optisch.
-       ================================================================ -->
-  <xacro:property name="oak_x"   value="0.120"/>
-  <xacro:property name="oak_y"   value="0.000"/>
-  <xacro:property name="oak_z"   value="0.360"/>
-  <xacro:property name="oak_yaw" value="0.000"/>
+       [GEMESSEN 26.07.2026] Aktuell verbaut: Luxonis OAK-D-S2 (Autofokus).
+       Geplant war OAK 4 D Pro Wide FF (derzeit nicht lieferbar) - beim
+       Wechsel diese Werte pruefen. MUSS mit der Montagepose in
+       robot_bringup/launch/oak.launch.py uebereinstimmen (dort haengt der
+       reale TF-Baum des Treibers dran)!
+       Gemessen: x=150 mm, mittig, 1340 mm ueber BODEN, 20 Grad nach unten.
+       z hier = 1.340 - 0.090 (base_link liegt 9 cm ueber dem Boden) = 1.250
+       ================================================================ -->
+  <xacro:property name="oak_x"     value="0.150"/>
+  <xacro:property name="oak_y"     value="0.000"/>
+  <xacro:property name="oak_z"     value="1.250"/>
+  <xacro:property name="oak_yaw"   value="0.000"/>
+  <xacro:property name="oak_pitch" value="0.349"/>  <!-- 20 Grad nach unten -->
+  <xacro:property name="oak_roll"  value="0.000"/>
   <!-- ================================================================
        SENSOR-MONTAGE: 2x VL53L7CX [ANPASSEN]
@@ -147,5 +156,5 @@
     <parent link="base_link"/>
     <child link="camera_link"/>
-    <origin xyz="${oak_x} ${oak_y} ${oak_z}" rpy="0 0 ${oak_yaw}"/>
+    <origin xyz="${oak_x} ${oak_y} ${oak_z}" rpy="${oak_roll} ${oak_pitch} ${oak_yaw}"/>
   </joint>
   <link name="camera_rgb_optical_frame"/>

Commit message: TF-Konflikte bereinigen: eindeutige Besitzer je Transform
Der HARDWARE_AKTIVIERUNGSPLAN des Kartenpakets verlangt genau einen Publisher
pro Transform und verbietet u.a. statisches map->odom parallel zu SLAM sowie
doppelte feste Sensor-TFs aus URDF und static_transform_publisher. Beides war
hier LATENT vorhanden: robot_state_publisher laeuft im produktiven Pfad noch
nicht, die Konflikte haetten also erst beim Start von SLAM bzw. der URDF-TFs
zugeschlagen.

1) URDF-VL53-Pose war veraltet und wich deutlich von der Messung ab:
     x 0.300 -> 0.290, y +/-0.110 -> +/-0.095, z 0.050 -> 0.215,
     Eindrehung -/+0.350 rad -> 0 (die Sensoren schauen gerade nach vorn).
   Der z-Fehler betrug 16.5 cm, der Winkelfehler 20 Grad. Ein
   robot_state_publisher haette damit eine falsche Sensorpose publiziert.
   URDF liefert jetzt exakt dieselbe Pose wie der statische Publisher
   (verifiziert: xacro erzeugt xyz="0.29 0.095 0.215" rpy 0).

2) vl53_near_field.launch.py: neues Argument publish_sensor_tf (Default true).
   Auf false setzen, sobald ein robot_state_publisher dieselben Frames aus der
   URDF liefert. Verifiziert: false -> 0 statische Publisher, true -> 2.

3) nav_real.launch.py: neues Argument static_map_odom (Default true). Das
   statische map->odom ist als Platzhalter gekennzeichnet und MUSS auf false,
   sobald RTAB-Map oder AMCL laeuft. Verifiziert: false -> Publisher bleibt weg,
   true -> Publisher startet.

Defaults bleiben unveraendert, der heutige Fahrbetrieb ist nicht betroffen.
Beide Schalter sind die Vorbereitung fuer die SLAM-Inbetriebnahme.

Co-Authored-By: Claude Opus 4.8 <noreply@anthropic.com>

File: src/robot_description/urdf/mobile_manipulator_dummy.urdf.xacro (robot description, xacro)
@@ -56,12 +56,18 @@
   <xacro:property name="oak_roll"  value="0.000"/>
   <!-- ================================================================
-       SENSOR-MONTAGE: 2x VL53L7CX [ANPASSEN]
-       Werte muessen spaeter zur real kalibrierten Montage passen.
-       left_y > 0 ist links. inward_yaw dreht beide Sensoren zur Mitte.
-       ================================================================ -->
-  <xacro:property name="vl53_x"          value="0.300"/>
-  <xacro:property name="vl53_y_abs"      value="0.110"/>
-  <xacro:property name="vl53_z"          value="0.050"/>
-  <xacro:property name="vl53_inward_yaw" value="0.350"/>  <!-- ca. 20 Grad -->
+       SENSOR-MONTAGE: 2x VL53L7CX
+       [GEMESSEN 24.07.2026 am aufgebauten Roboter] left_y > 0 ist links.
+       MUSS mit den statischen TFs in vl53_near_field/launch/vl53_near_field.launch.py
+       uebereinstimmen - dort haengt die reale TF-Kette dran. Wenn hier und dort
+       verschiedene Posen stehen und beide Quellen laufen, streiten zwei Publisher
+       um denselben Transform.
+       Gemessen: 290 mm vor der Antriebsrad-Achse, +/-95 mm von der Mittellinie,
+       305 mm ueber BODEN -> z = 0.305 - 0.090 = 0.215 ueber base_link.
+       KEINE Eindrehung: beide Sensoren schauen gerade nach vorn.
+       ================================================================ -->
+  <xacro:property name="vl53_x"          value="0.290"/>
+  <xacro:property name="vl53_y_abs"      value="0.095"/>
+  <xacro:property name="vl53_z"          value="0.215"/>
+  <xacro:property name="vl53_inward_yaw" value="0.000"/>  <!-- geradeaus, nicht eingedreht -->
   <!-- ================================================================
        ARM-MONTAGE / DUMMY-LINKLAENGEN [ANPASSEN]

Commit message: OAK-Neigung nachgemessen: 18.94 statt 20.0 Grad
Aus der Bodenebene der Punktwolke bestimmt (reine Messung, Roboter stand):
mit den eingetragenen 20.0 Grad stieg der gemessene Boden ueber die
Entfernung an - -0.083 m bei 1.5 m und -0.064 m bei 2.5 m statt konstant
-0.090 m. Das entspricht 1.06 Grad Neigungsfehler. Wert in oak.launch.py und
URDF auf 0.3306 rad (18.94 Grad) korrigiert.

WICHTIG - meine Arbeitshypothese war FALSCH: Ich hatte vermutet, die dicken
Hindernisbaender in der Karte kaemen daher, dass entfernter Boden faelschlich
als Hindernis eingetragen wird. Das ist widerlegt:
  - der Hoehenfehler betraegt nur 26 mm auf 2.5 m, die Bodenschwelle liegt
    bei 150 mm - viel zu wenig fuer eine Fehlklassifikation;
  - gemessene Hoehenverteilung im Kartierbereich (<2.5 m): 66.5 % der Punkte
    sind Boden (<5 cm) und werden korrekt ausgefiltert, 29.1 % liegen
    tatsaechlich auf Hindernishoehe (15-150 cm).
Die 29.1 % decken sich mit den 30.7 % belegten Zellen der Karte. Die Karte
bildet also den real vollgestellten Raum korrekt ab (Kartons, Taschen, Stuhl,
Schreibtisch) - sie war nicht fehlerhaft.

Vorbehalt zur Neigung: ein Teil des 1-Grad-Werts kann echte Bodenneigung im
Raum sein, nicht Montagefehler. Die Korrektur ist klein und risikolos.

Co-Authored-By: Claude Opus 4.8 <noreply@anthropic.com>

File: src/robot_description/urdf/mobile_manipulator_dummy.urdf.xacro (robot description, xacro)
@@ -46,6 +46,8 @@
        robot_bringup/launch/oak.launch.py uebereinstimmen (dort haengt der
        reale TF-Baum des Treibers dran)!
-       Gemessen: x=150 mm, mittig, 1340 mm ueber BODEN, 20 Grad nach unten.
+       Gemessen: x=150 mm, mittig, 1340 mm ueber BODEN, ca. 20 Grad nach unten.
        z hier = 1.340 - 0.090 (base_link liegt 9 cm ueber dem Boden) = 1.250
+       Neigung am 27.07.2026 aus der Bodenebene nachgemessen: 18.94 statt
+       20.0 Grad (siehe oak_pitch unten und oak.launch.py).
        ================================================================ -->
   <xacro:property name="oak_x"     value="0.150"/>
@@ -53,5 +55,5 @@
   <xacro:property name="oak_z"     value="1.250"/>
   <xacro:property name="oak_yaw"   value="0.000"/>
-  <xacro:property name="oak_pitch" value="0.349"/>  <!-- 20 Grad nach unten -->
+  <xacro:property name="oak_pitch" value="0.3306"/> <!-- 18.94 Grad, nachgemessen 27.07.2026 -->
   <xacro:property name="oak_roll"  value="0.000"/>
   <!-- ================================================================
