Commit message: fix: vermessenen Footprint für Wohnungstüren anwenden
Die gemessene Plattform ist mit 460 mm deutlich schmaler und mit 270/110 mm asymmetrischer als das bisherige 700x500-mm-Modell. Nav2, Explorer und URDF verwenden jetzt die sichere Hülle einschließlich VL53-Überstand; bei der 680-mm-Tür bleiben lokal 90 mm je Seite.\n\nMotorlos verifiziert: 49 registrierte Tests, identische Nav2-/Kollisionspolygone und ein gerader erfolgreicher NavFn-Pfad durch eine synthetische 690-mm-Tür bei 0 rpm. Rückfall bleibt der konservative 0,40-m-Kreis beziehungsweise active_drive=false.

File: src/robot_description/urdf/mobile_manipulator_dummy.urdf.xacro (robot description, xacro)
@@ -21,10 +21,14 @@
 <robot xmlns:xacro="http://www.ros.org/wiki/xacro" name="mobile_pick_place_dummy">
   <!-- ================================================================
-       BASIS-MASSE [ANPASSEN]
+       BASIS-MASSE [GEMESSEN 18.08.2026]
        Koordinaten: x vorne, y links, z oben. base_footprint liegt am Boden.
-       base_link liegt im geometrischen Zentrum der Chassis-Box.
-       ================================================================ -->
-  <xacro:property name="base_length" value="0.70"/>    <!-- [m] Plattformlaenge -->
-  <xacro:property name="base_width"  value="0.50"/>    <!-- [m] Plattformbreite -->
+       base_link liegt in der Antriebsachse, mittig zwischen den Raedern.
+       Chassis: 270 mm vor und 110 mm hinter base_link, maximal 460 mm breit;
+       die vordere Stirn ist 360 mm breit. Die Vorderecken sind abgeschraegt;
+       ohne gemessene Schraegentiefe ist die Box ihre sichere Huelle.
+       ================================================================ -->
+  <xacro:property name="base_length" value="0.38"/>    <!-- [m] Chassislaenge -->
+  <xacro:property name="base_width"  value="0.46"/>    <!-- [m] maximale Breite -->
+  <xacro:property name="base_center_x" value="0.08"/>  <!-- (0.270 - 0.110) / 2 -->
   <xacro:property name="base_height" value="0.18"/>    <!-- [m] Plattformhoehe -->
   <!-- ================================================================
@@ -137,8 +141,10 @@
   <link name="base_link">
     <visual>
+      <origin xyz="${base_center_x} 0 0" rpy="0 0 0"/>
       <geometry><box size="${base_length} ${base_width} ${base_height}"/></geometry>
       <material name="mat_base"/>
     </visual>
     <collision>
+      <origin xyz="${base_center_x} 0 0" rpy="0 0 0"/>
       <geometry><box size="${base_length} ${base_width} ${base_height}"/></geometry>
     </collision>
